Commit message: All the 6 motors working in the real robot

File: epos_hardware/robot/hexapodo_velocity.urdf (robot description, URDF)
Before this commit: robot example, 12 links, 6 joints
Links:
- removed link link11
- removed link link12
- removed link link21
- removed link link22
- removed link link31
- removed link link32
- removed link link41
- removed link link42
- removed link link51
- removed link link52
- removed link link61
- removed link link62
- added link chassis, mass 5.771; collision mesh filename=package://epos_hardware/robot/caja.stl scale=0.001 0.001 0.001; visual mesh filename=package://rhex_description/meshes/caja.stl scale=0.001 0.001 0.001
- added link leg_1, mass 0.057; visual mesh filename=package://epos_hardware/robot/pvc.stl scale=0.001 0.001 0.001
- added link leg_2, mass 0.057; visual mesh filename=package://epos_hardware/robot/pvc.stl scale=0.001 0.001 0.001
- added link leg_3, mass 0.057; visual mesh filename=package://epos_hardware/robot/pvc.stl scale=0.001 0.001 0.001
- added link leg_4, mass 0.057; visual mesh filename=package://epos_hardware/robot/pvc.stl scale=0.001 0.001 0.001
- added link leg_5, mass 0.057; visual mesh filename=package://epos_hardware/robot/pvc.stl scale=0.001 0.001 0.001
- added link leg_6, mass 0.057; visual mesh filename=package://epos_hardware/robot/pvc.stl scale=0.001 0.001 0.001
Joints:
- removed joint test_joint
- removed joint test_joint2
- removed joint test_joint3
- removed joint test_joint4
- removed joint test_joint5
- removed joint test_joint6
- added joint joint_1: type revolute, parent chassis, child leg_1
- added joint joint_2: type revolute, parent chassis, child leg_2, limit lower=-10000.0 upper=10000.0 effort=3.5 velocity=38.0
- added joint joint_3: type revolute, parent chassis, child leg_3, limit lower=-10000.0 upper=10000.0 effort=3.5 velocity=38.0
- added joint joint_4: type revolute, parent chassis, child leg_4, limit lower=-10000.0 upper=10000.0 effort=3.5 velocity=38.0
- added joint joint_5: type revolute, parent chassis, child leg_5, limit lower=-10000.0 upper=10000.0 effort=3.5 velocity=38.0
- added joint joint_6: type revolute, parent chassis, child leg_6, limit lower=-10000.0 upper=10000.0 effort=3.5 velocity=38.0
